File: PCB/Plonke.kicad_sch (KiCad schematic)
At the start: 17 parts, among them J1 USB_C_Receptacle_USB2.0_16P, J2 AVR-ISP-6, U1 ATmega32U4-A, U2 USB6B1, Y1 Crystal_GND24_Small

Commit message: tim plz help me
many many changes
Parts:
- removed C1: 100nF, Capacitor_THT:C_Disc_D4.7mm_W2.5mm_P5.00mm, symbol Device:C
- removed C4: 1u, Capacitor_THT:C_Disc_D4.7mm_W2.5mm_P5.00mm, symbol Device:C
- removed U1: ATmega32U4-A, Package_QFP:TQFP-44_10x10mm_P0.8mm, symbol MCU_Microchip_ATmega:ATmega32U4-A
- added BTN2: Boot, Button_Switch_THT:SW_PUSH_6mm, symbol Switch:SW_Push
- added C1: 4.7u, Capacitor_THT:CP_Radial_D4.0mm_P1.50mm, symbol Device:C_Polarized
- added D48, D49: LED, LED_THT:LED_D3.0mm, symbol Device:LED
- added R6, R7, R8: 1.5k, Resistor_THT:R_Axial_DIN0207_L6.3mm_D2.5mm_P10.16mm_Horizontal, symbol Device:R
- added U3: ATmega328-P, Package_DIP:DIP-28_W7.62mm, symbol MCU_Microchip_ATmega:ATmega328-P
- BTN1: value SW_Push -> Reset
- C5, C6: value 12pF -> 20pF
- J2: footprint Connector_PinHeader_2.54mm:PinHeader_2x03_P2.54mm_Horizontal -> Connector_PinHeader_2.54mm:PinHeader_2x03_P2.54mm_Vertical
Connections:
- net SCL is gone; now on net R2: J2.3 (SCK)
- net C1: now also U3.14 (PB0)
- net C10: now also U3.26 (PC3)
- net C11: now also U3.3 (PD1)
- net C12: now also U3.2 (PD0)
- net C2: now also U3.13 (PD7)
- net C3: now also U3.12 (PD6)
- net C4: now also BTN2.2, U3.11 (PD5)
- net C5: now also U3.16 (PB2)
- net C6: now also U3.15 (PB1)
- net C7: now also U3.23 (PC0)
- net C8: now also U3.24 (PC1)
- net C9: now also U3.25 (PC2)
- net GND: now also BTN2.1, C1.2, D48.1 (K), D49.1 (K), U3.22 (GND), U3.8 (GND)
- net MISO: now also U3.18 (PB4)
- net MOSI: now also U3.17 (PB3)
- net R2: now also U3.19 (PB5)
- net R4: now also U3.6 (PD4)
- net RESET: now also U3.1 (~{RESET}/PC6)
- net VBUS: now also C1.1, R8.1, U3.20 (AVCC), U3.7 (VCC)
- net at C5.2, Y1.3: now also U3.9 (XTAL1/PB6)
- net at C6.2, Y1.1: now also U3.10 (XTAL2/PB7)
- net at R2.2: now also U3.5 (PD3)
- net at R3.2: now also U3.4 (PD2)
- net at J1.A7 (D-), J1.B7 (D-), U2.2 (I/O1): now also R8.2
- new net: D49.2 (A), R7.2
- new net: R7.1, U3.28 (PC5)
- new net: D48.2 (A), R6.2
- new net: R6.1, U3.27 (PC4)
- no-connect marks 3 -> 4
Other:
- moved on the sheet: BTN1, C5, C6, R1, R2, R3, U2, Y1
