File: PCB/Plonke.kicad_pcb (KiCad board)
At the start: 2 copper layers, 232 x 101 mm, 116 parts, among them J1 USB_C_Receptacle_USB2.0_16P, J2 AVR-ISP-6, SW1 SW_Push, SW10 SW_Push, SW11 SW_Push, SW12 SW_Push, SW13 SW_Push, SW14 SW_Push, SW15 SW_Push, SW16 SW_Push, SW17 SW_Push, SW18 SW_Push, SW19 SW_Push, SW2 SW_Push, SW20 SW_Push, SW21 SW_Push, SW22 SW_Push, SW23 SW_Push, SW24 SW_Push, SW25 SW_Push, SW26 SW_Push, SW27 SW_Push, SW28 SW_Push, SW29 SW_Push, SW3 SW_Push, SW30 SW_Push, SW31 SW_Push, SW32 SW_Push, SW33 SW_Push, SW34 SW_Push, SW35 SW_Push, SW36 SW_Push, SW37 SW_Push, SW38 SW_Push, SW39 SW_Push, SW4 SW_Push, SW40 SW_Push, SW41 SW_Push, SW42 SW_Push, SW43 SW_Push, SW44 SW_Push, SW45 SW_Push, SW46 SW_Push, SW47 SW_Push, SW5 SW_Push, SW6 SW_Push, SW7 SW_Push, SW8 SW_Push, SW9 SW_Push, U1 ATmega32U4-A, U2 USB6B1, Y1 Crystal_GND24_Small

Commit message: tim plz help me
many many changes
Parts:
- removed U1: ATmega32U4-A, Package_QFP:TQFP-44_10x10mm_P0.8mm
- added BTN2: Boot, Button_Switch_THT:SW_PUSH_6mm, F.Cu at (170.4, 56.2)
- added D48: LED, LED_THT:LED_D3.0mm, F.Cu at (175.8, 49.8)
- added D49: LED, LED_THT:LED_D3.0mm, F.Cu at (171.0, 49.8)
- added R6: 1.5k, Resistor_THT:R_Axial_DIN0207_L6.3mm_D2.5mm_P10.16mm_Horizontal, F.Cu at (163.9, 67.6)
- added R7: 1.5k, Resistor_THT:R_Axial_DIN0207_L6.3mm_D2.5mm_P10.16mm_Horizontal, F.Cu at (160.6, 67.5)
- added R8: 1.5k, Resistor_THT:R_Axial_DIN0207_L6.3mm_D2.5mm_P10.16mm_Horizontal, F.Cu at (138.1, 57.0)
- added REF**: MountingHole_3.2mm_M3, MountingHole:MountingHole_3.2mm_M3, F.Cu at (251.5, 57.6)
- added REF**: MountingHole_3.2mm_M3, MountingHole:MountingHole_3.2mm_M3, F.Cu at (48.7, 39.9)
- added U3: ATmega328-P, Package_DIP:DIP-28_W7.62mm, F.Cu at (154.9, 59.9)
- BTN1: value SW_Push -> Reset
- C1: value 100nF -> 4.7u; footprint Capacitor_THT:C_Disc_D4.7mm_W2.5mm_P5.00mm -> Capacitor_THT:CP_Radial_D4.0mm_P1.50mm
- C5, C6: value 12pF -> 20pF
- R2: moved to B.Cu
- moved R1 105.0 mm to (182.8, 66.5), turned to 0 degrees
- moved C1 52.4 mm to (120.0, 49.9), turned to 0 degrees
- moved R2 40.4 mm to (134.7, 49.0), turned to 180 degrees
- moved R3 38.7 mm to (134.7, 45.8)
- moved C4 34.4 mm to (115.5, 46.2), turned to 180 degrees
- moved R5 31.8 mm to (170.1, 67.1), turned to 0 degrees
- moved C6 25.2 mm to (132.3, 51.7), turned to -90 degrees
- moved J2 22.0 mm to (180.4, 60.6)
- moved C5 19.9 mm to (135.3, 51.7), turned to -90 degrees
- moved R4 16.0 mm to (170.1, 63.9), turned to 0 degrees
- moved D7 13.9 mm to (188.9, 61.0)
- moved D19 13.3 mm to (190.2, 55.6)
- moved D31 11.8 mm to (190.4, 50.2)
- moved BTN1 11.0 mm to (157.3, 49.9)
- moved D32 9.70 mm to (202.0, 55.6)
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Connections:
- D1 pad 1: R1 -> MISO
- D10 pad 1: R1 -> MISO
- D11 pad 1: R1 -> MISO
- D12 pad 1: R1 -> MISO
- D2 pad 1: R1 -> MISO
- D25 pad 1: R3 -> MOSI
- D26 pad 1: R3 -> MOSI
- D27 pad 1: R3 -> MOSI
- D28 pad 1: R3 -> MOSI
- D29 pad 1: R3 -> MOSI
- D3 pad 1: R1 -> MISO
- D30 pad 1: R3 -> MOSI
- D31 pad 1: R3 -> MOSI
- D32 pad 1: R3 -> MOSI
- D33 pad 1: R3 -> MOSI
- D34 pad 1: R3 -> MOSI
- D35 pad 1: R3 -> MOSI
- D36 pad 1: R3 -> MOSI
- D4 pad 1: R1 -> MISO
- D5 pad 1: R1 -> MISO
- D6 pad 1: R1 -> MISO
- D7 pad 1: R1 -> MISO
- D8 pad 1: R1 -> MISO
- D9 pad 1: R1 -> MISO
- J2 pad 3: SCL -> R2
Routing:
- net R1: track 270.7 -> 0.00 mm, vias 4 -> 0
- net R4: track 251.8 -> 0.00 mm, vias 3 -> 0
- net R3: track 249.9 -> 0.00 mm, vias 4 -> 0
- net R2: track 245.2 -> 0.00 mm, vias 4 -> 0
- net C1: track 208.1 -> 0.00 mm, vias 5 -> 0
- net C2: track 192.6 -> 0.00 mm, vias 5 -> 0
- net C12: track 187.9 -> 0.00 mm, vias 3 -> 0
- net C3: track 173.7 -> 0.00 mm, vias 5 -> 0
- net C11: track 167.0 -> 0.00 mm, vias 3 -> 0
- net C10: track 145.0 -> 0.00 mm, vias 3 -> 0
- net C4: track 136.6 -> 0.00 mm, vias 3 -> 0
- net C8: track 130.5 -> 0.00 mm, vias 1 -> 0
- net C9: track 120.2 -> 0.00 mm, vias 3 -> 0
- net C5: track 118.0 -> 0.00 mm, vias 3 -> 0
- net GND: track 116.5 -> 0.00 mm, vias 1 -> 0
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Other:
- board size 232 x 101 mm -> 232 x 103.5 mm

Commit message: i did this
Parts:
- moved REF** 18.6 mm to (48.5, 58.5)
- moved C4 14.9 mm to (114.0, 61.0), turned to -90 degrees
- moved C6 11.2 mm to (121.5, 55.0), turned to 0 degrees
- moved D42 10.8 mm to (106.2, 66.3)
- moved Y1 9.57 mm to (114.5, 49.0), turned to -90 degrees
- moved D41 9.27 mm to (94.2, 66.3)
- moved R1 8.16 mm to (191.0, 66.2)
- moved D40 7.72 mm to (82.2, 66.3)
- moved D38 7.26 mm to (58.2, 66.3)
- moved D8 6.67 mm to (205.0, 66.2)
- moved D30 6.58 mm to (108.9, 61.0)
- moved D39 6.17 mm to (70.2, 66.3)
- moved D6 6.16 mm to (106.4, 50.0)
- moved D9 5.79 mm to (217.2, 66.2)
- moved D29 5.49 mm to (96.4, 61.0)
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Routing:
- net R2: track 0.00 -> 237.8 mm
- net MOSI: track 0.00 -> 237.2 mm
- net R4: track 0.00 -> 225.5 mm
- net MISO: track 0.00 -> 164.3 mm
- net Net-(D43-A): track 0.00 -> 132.9 mm
- net Net-(D44-A): track 0.00 -> 124.6 mm
- net Net-(D42-A): track 0.00 -> 118.7 mm
- net Net-(D45-A): track 0.00 -> 117.9 mm
- net Net-(D46-A): track 0.00 -> 111.0 mm
- net Net-(D41-A): track 0.00 -> 106.7 mm
- net Net-(D47-A): track 0.00 -> 105.2 mm
- net Net-(D32-A): track 0.00 -> 101.8 mm
- net Net-(D31-A): track 0.00 -> 98.5 mm
- net Net-(D40-A): track 0.00 -> 98.5 mm
- net Net-(D30-A): track 0.00 -> 94.5 mm
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